Commit message: Added Config and Robot file for updated urdf
and fixed urdf to help with running the code

File: Chess/backend/KoalbyHumanoid/Simulation Files/Humanoid_URDF_9-10/urdf/Humanoid_URDF_9-10.urdf (robot description, URDF)
Before this commit: robot Humanoid_URDF_9-10, 28 links, 27 joints
Joints:
- joint abdominalcrunch: type continuous -> revolute
- joint ankle_left: type continuous -> revolute
- joint ankle_right: type continuous -> revolute
- joint biceplift_left: type continuous -> revolute
- joint biceplift_right: type continuous -> revolute
- joint chestturn: type continuous -> revolute
- joint elbow_left: type continuous -> revolute
- joint elbow_right: type continuous -> revolute
- joint gripper_left: type continuous -> revolute
- joint gripper_right: type continuous -> revolute
- joint handcurl_left: type continuous -> revolute
- joint handcurl_right: type continuous -> revolute
- joint headnod: type continuous -> revolute
- joint hiplift_left: type continuous -> revolute
- joint hiplift_right: type continuous -> revolute
- joint hiprotate_left: type continuous -> revolute
- joint hiprotate_right: type continuous -> revolute
- joint knee_left: type continuous -> revolute
- joint knee_right: type continuous -> revolute
- joint neckturn: type continuous -> revolute
- joint shoulderspin_left: type continuous -> revolute
- joint shoulderspin_right: type continuous -> revolute
- joint thighlift_left: type continuous -> revolute
- joint thighlift_right: type continuous -> revolute
- joint waistlean: type continuous -> revolute
- joint wristspin_left: type continuous -> revolute
- joint wristspin_right: type continuous -> revolute

Commit message: joint limits and arm tests

File: Chess/backend/KoalbyHumanoid/Simulation Files/Humanoid_URDF_9-10/urdf/Humanoid_URDF_9-10.urdf (robot description, URDF)
Before this commit: robot Humanoid_URDF_9-10, 28 links, 27 joints
Joints:
- joint biceplift_left: limit (none) -> lower=-1.22173 upper=1.5708
- joint biceplift_right: limit (none) -> lower=-1.22173 upper=1.5708
- joint elbow_left: limit (none) -> lower=-1.74533 upper=1.74533
- joint gripper_left: limit (none) -> lower=0 upper=0.698132
- joint gripper_right: limit (none) -> lower=0 upper=0.698132
- joint handcurl_left: limit (none) -> lower=-2.00713 upper=2.00713
- joint handcurl_right: limit (none) -> lower=-2.00713 upper=2.00713
- joint shoulderspin_left: limit (none) -> lower=-1.5708 upper=1.5708
- joint shoulderspin_right: limit (none) -> lower=-1.5708 upper=1.5708
- joint wristspin_left: limit (none) -> lower=-1.5708 upper=1.5708
- joint wristspin_right: limit (none) -> lower=-1.5708 upper=1.5708
