Commit message: Changed my pick and place code to a class structure

File: Chess/backend/Testing/FinleyJNEWARMS_2024_straight_4.urdf (robot description, URDF)
Before this commit: robot FinleyJNEWARMS_2024_straight_4, 31 links, 30 joints
Joints:
- joint elbow_right: limit lower=0 upper=0 effort=0 velocity=0 -> (none)
- joint forearm_right: limit lower=0 upper=0 effort=0 velocity=0 -> (none)
- joint hand_right: limit lower=0 upper=0 effort=0 velocity=0 -> (none)
- joint shoulder1_right: limit lower=0 upper=0 effort=0 velocity=0 -> (none)
- joint shoulder2_right: limit lower=0 upper=0 effort=0 velocity=0 -> (none)
- joint wrist_right: limit lower=0 upper=0 effort=0 velocity=0 -> (none)
